File: sensors.kicad_sch (KiCad schematic)
At the start: 15 parts, among them U4 ICM42605, U5 MMC5983MA, U6 ICP20100

Commit message: draft: schematic and layout for H20R1
Changed lines of the file:
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@@
     (effects (font (size 1.27 1.27)) (justify left bottom))
   )
-  (text "Pullup values chosen\nas per Pixhawk standards" (at 228.6 81.28 0)
+  (text "Pullup values chosen\nas per Pixhawk standards" (at 222.25 74.93 0)
     (effects (font (size 1.27 1.27)) (justify left bottom))
   )

Commit message: replace sdio with spi2, finish routing, front silkscreen
Parts:
- R23, R7: footprint Resistor_SMD:R_0402_1005Metric -> Resistor_SMD:R_0201_0603Metric
